Commit message: feat(simulation): add chassis contact physics and drop validation
Add 25 primitive collisions and initial ODE friction/contact settings.
Aggregate fixed-component masses and tensors with frame rotations and the
parallel-axis theorem, retaining massless-part geometry. Generate a passive
three-body scene with two free wheels and the unchanged 0.877 kg subtotal.

Provide an isolated ground-contact launch, state-based drop validator,
conservation/transform/surface tests and bilingual operating instructions.
Install the Python generator and add NumPy to test/build dependencies.

Validation: isolated staged tree passes repository checks, 11 unit tests,
description/bringup builds and SDF validation. Previously recorded local
drop testing confirmed all four supports contact the floor and settle.
Friction values are initial estimates; driven motion is added separately.

File: src/odin_racer/racer_description/urdf/motor_assembly.xacro (robot description, xacro)
@@ -52,4 +52,8 @@
         <material name="motor_metal"/>
       </visual>
+      <collision name="${side}_gearbox_envelope_collision">
+        <origin xyz="${motor_axis_offset/2} ${-sign*assumed_gearbox_depth/2} 0"/>
+        <geometry><box size="${gearbox_length} ${assumed_gearbox_depth} ${gearbox_height}"/></geometry>
+      </collision>
       <visual name="motor_can">
         <origin xyz="${motor_axis_offset} ${-sign*(assumed_gearbox_depth+can_depth/2)} 0" rpy="${pi/2} 0 0"/>
@@ -57,4 +61,8 @@
         <material name="motor_metal"/>
       </visual>
+      <collision name="${side}_motor_can_collision">
+        <origin xyz="${motor_axis_offset} ${-sign*(assumed_gearbox_depth+can_depth/2)} 0" rpy="${pi/2} 0 0"/>
+        <geometry><cylinder radius="${motor_diameter/2}" length="${can_depth}"/></geometry>
+      </collision>
       <visual name="gmr_cover">
         <origin xyz="${motor_axis_offset} ${-sign*(motor_total_depth-assumed_encoder_depth/2)} 0" rpy="${pi/2} 0 0"/>
@@ -62,4 +70,8 @@
         <material name="motor_black"/>
       </visual>
+      <collision name="${side}_gmr_cover_collision">
+        <origin xyz="${motor_axis_offset} ${-sign*(motor_total_depth-assumed_encoder_depth/2)} 0" rpy="${pi/2} 0 0"/>
+        <geometry><cylinder radius="${encoder_diameter/2}" length="${assumed_encoder_depth}"/></geometry>
+      </collision>
     </link>
     <joint name="${side}_motor_mount" type="fixed">
@@ -79,4 +91,8 @@
         <material name="motor_black"/>
       </visual>
+      <collision name="${side}_vertical_web_collision">
+        <origin xyz="${motor_axis_offset/2} ${sign*assumed_bracket_thickness/2} ${(plate_bottom_z-gearbox_height/2)/2}"/>
+        <geometry><box size="${assumed_bracket_length} ${assumed_bracket_thickness} ${bracket_height}"/></geometry>
+      </collision>
       <visual name="top_flange">
         <origin xyz="${motor_axis_offset/2} ${sign*(assumed_bracket_thickness-assumed_bracket_reach/2)} ${plate_bottom_z-assumed_bracket_thickness/2}"/>
@@ -84,4 +100,8 @@
         <material name="motor_black"/>
       </visual>
+      <collision name="${side}_top_flange_collision">
+        <origin xyz="${motor_axis_offset/2} ${sign*(assumed_bracket_thickness-assumed_bracket_reach/2)} ${plate_bottom_z-assumed_bracket_thickness/2}"/>
+        <geometry><box size="${assumed_bracket_length} ${assumed_bracket_reach} ${assumed_bracket_thickness}"/></geometry>
+      </collision>
     </link>
     <joint name="${side}_motor_bracket_mount" type="fixed">
@@ -96,4 +116,8 @@
         <material name="motor_metal"/>
       </visual>
+      <collision name="${side}_output_shaft_collision">
+        <origin xyz="0 ${sign*(outer_y+shaft_length/2-wheel_track/2)} 0" rpy="${pi/2} 0 0"/>
+        <geometry><cylinder radius="${shaft_diameter/2}" length="${shaft_length}"/></geometry>
+      </collision>
     </link>
     <joint name="${side}_output_shaft_mount" type="fixed">

File: src/odin_racer/racer_description/urdf/odin1.xacro (robot description, xacro)
@@ -12,4 +12,9 @@
         <material name="odin_shell"><color rgba="0.16 0.18 0.20 1"/></material>
       </visual>
+      <!-- Full CAD bounds, including connectors; conservative solid envelope. -->
+      <collision name="odin_body_collision">
+        <origin xyz="-0.0036 0 0.031"/>
+        <geometry><box size="0.0464 0.100 0.062"/></geometry>
+      </collision>
       <!-- Estimated uniform body box COM/inertia; manufacturer's mass only.
            Body CAD depth -3..40 mm; hole-group midpoint depth 20.4 mm. -->

File: src/odin_racer/racer_description/urdf/robot.urdf.xacro (robot description, xacro)
@@ -1,4 +1,6 @@
 <?xml version="1.0"?>
-<!-- CAD-based geometry and approximate inertias for preview; no contact or drive simulation. -->
+<!-- CAD plate and user-specified wheel/ball geometry.
+     Preview with approximate inertias and primitive collisions. The dedicated
+     contact-world generator adds physics; no drive or measured calibration. -->
 <robot xmlns:xacro="http://www.ros.org/wiki/xacro" name="odin_racer_preview">
   <!-- SI units. Dimensions reported by the user; level plate height is a
@@ -7,4 +9,14 @@
   <xacro:property name="plate_length" value="0.24741600036621094"/>
   <xacro:property name="plate_height" value="0.062"/>
+  <!-- Collision envelopes measured from the STL in its local frame.
+       The slab fills cutouts; the upper box conservatively fills space between
+       raised CAD features. Neither is machining or self-collision geometry. -->
+  <xacro:property name="plate_width" value="0.220"/>
+  <xacro:property name="plate_thickness" value="0.0035"/>
+  <xacro:property name="plate_upper_min_x" value="-0.11904653906822205"/>
+  <xacro:property name="plate_upper_max_x" value="0.07495316863059998"/>
+  <xacro:property name="plate_upper_min_y" value="-0.07358216494321823"/>
+  <xacro:property name="plate_upper_max_y" value="0.10356252640485764"/>
+  <xacro:property name="plate_upper_top" value="0.0335"/>
   <xacro:property name="wheel_radius" value="0.03325"/>
   <!-- User-adopted tire + hub mass, kg. Fasteners ignored by instruction. -->
@@ -45,4 +57,12 @@
       <material name="body"/>
     </visual>
+    <collision name="plate_slab_collision">
+      <origin xyz="${plate_center_x} 0 ${plate_bottom_z+plate_thickness/2}"/>
+      <geometry><box size="${plate_length} ${plate_width} ${plate_thickness}"/></geometry>
+    </collision>
+    <collision name="plate_raised_envelope_collision">
+      <origin xyz="${plate_center_x+(plate_upper_min_x+plate_upper_max_x)/2} ${(plate_upper_min_y+plate_upper_max_y)/2} ${plate_bottom_z+(plate_thickness+plate_upper_top)/2}"/>
+      <geometry><box size="${plate_upper_max_x-plate_upper_min_x} ${plate_upper_max_y-plate_upper_min_y} ${plate_upper_top-plate_thickness}"/></geometry>
+    </collision>
   </link>
   <xacro:macro name="drive_wheel" params="side y">
@@ -62,4 +82,8 @@
         <material name="rubber"/>
       </visual>
+      <collision name="${side}_wheel_collision">
+        <origin rpy="${pi/2} 0 0"/>
+        <geometry><cylinder radius="${wheel_radius}" length="${wheel_width}"/></geometry>
+      </collision>
     </link>
     <joint name="${side}_wheel_joint" type="continuous">
@@ -81,4 +105,9 @@
         <material name="brass"/>
       </visual>
+      <!-- Circumscribed cylinder around the hex; top remains at mount Z=0. -->
+      <collision name="${side}_${end}_pillar_collision">
+        <origin xyz="0 0 ${-pillar_length/2}"/>
+        <geometry><cylinder radius="${pillar_width/sqrt(3)}" length="${pillar_length}"/></geometry>
+      </collision>
     </link>
     <joint name="${side}_${end}_pillar_mount_joint" type="fixed">
@@ -93,6 +122,6 @@
   <xacro:pillar_pair side="left" y="${ball_track/2}"/>
   <xacro:pillar_pair side="right" y="${-ball_track/2}"/>
-  <!-- Ball transfers, not swivel casters. Fixed visual spheres;
-       no rolling or friction model yet.
+  <!-- Ball transfers, not swivel casters. Fixed spheres with collision geometry;
+       contact-world generation adds low-friction sliding, not ball rotation.
        Housing is an envelope; flange
        width/thickness and hole diameters are absent from the product drawing.
@@ -113,4 +142,7 @@
       </inertial>
       <visual><geometry><sphere radius="${ball_radius}"/></geometry><material name="steel"/></visual>
+      <collision name="${side}_ball_collision">
+        <geometry><sphere radius="${ball_radius}"/></geometry>
+      </collision>
       <visual>
         <origin xyz="0 0 ${caster_height-ball_radius-housing_height/2}"/>
@@ -118,4 +150,8 @@
         <material name="steel"/>
       </visual>
+      <collision name="${side}_ball_housing_collision">
+        <origin xyz="0 0 ${caster_height-ball_radius-housing_height/2}"/>
+        <geometry><cylinder radius="${housing_radius}" length="${housing_height}"/></geometry>
+      </collision>
     </link>
     <joint name="front_${side}_caster_mount" type="fixed">
